Commit message: LiDAR now shows up and camera is in place. I don't understand why can't I use my own .stl file- even when it's just a copy of the existing hokuyo_10_ust.stl file, but for now it will have to do using the hokuyo_10_ust.stl file in place of the lds LiDAR model.

File: husky_description/urdf/accessories/ae_lidar.urdf.xacro (robot description, xacro)
@@ -58,5 +58,6 @@
         <geometry>
           <!-- Origin of this mesh is the base of the bracket. -->
-          <mesh filename="package://husky_description/meshes/accessories/lds.stl" />
+          <!--mesh filename="package://husky_description/meshes/accessories/lds.stl" /-->
+          <mesh filename="package://husky_description/meshes/accessories/hokuyo_ust10.stl" />
         </geometry>
         <material name="dark_grey" />

File: husky_description/urdf/cameras_and_lidars.urdf.xacro (robot description, xacro)
@@ -7,10 +7,10 @@
   <!-- Camera -->
   <xacro:simple_camera camera_name="sim_camera1" parent_link="top_plate_link" >
-    <origin xyz="0.16 0.16 0.16" rpy="0 0 0" />
+    <origin xyz="0.0 0.0 0.54" rpy="0 0 0" />
   </xacro:simple_camera>
   <!-- LiDAR -->
   <xacro:if value="$(arg ae_lidar_enabled)">
     <xacro:ae_lidar_mount topic="/scan" prefix="ae_lidar1" parent_link="top_plate_link">
-        <origin xyz="0.0 0.0 0.0" rpy="0 0 0" />
+        <origin xyz="0.32 0.0 0.0" rpy="0 0 0" />
       </xacro:ae_lidar_mount>
   </xacro:if>
